File: pcb/MacroMax703_pcb.kicad_pcb (KiCad board)
At the start: 2 copper layers, 99 x 49 mm, 21 parts, among them SW1 SW_Push, SW10 RotaryEncoder_Switch, SW11 RotaryEncoder_Switch, SW2 SW_Push, SW3 SW_Push, SW4 SW_Push, SW5 SW_Push, SW6 SW_Push, SW7 SW_Push, SW8 SW_Push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

Commit message: update pcb and firmware
Other:
- board text added: "MACROMAX703"
Changed lines of the file:
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@@
 			(plot_on_all_layers_selection 0x00000000_00000000_00000000_00000000)
 			(disableapertmacros no)
-			(usegerberextensions no)
-			(usegerberattributes yes)
-			(usegerberadvancedattributes yes)
-			(creategerberjobfile yes)
+			(usegerberextensions yes)
+			(usegerberattributes no)
+			(usegerberadvancedattributes no)
+			(creategerberjobfile no)
 			(dashed_line_dash_ratio 12)
 			(dashed_line_gap_ratio 3)
@@
 			(sketchdnponfab yes)
 			(crossoutdnponfab yes)
-			(subtractmaskfromsilk no)
+			(subtractmaskfromsilk yes)
 			(outputformat 1)
 			(mirror no)
-			(drillshape 1)
+			(drillshape 0)
 			(scaleselection 1)
-			(outputdirectory "")
+			(outputdirectory "../../gerbers/")
 		)
 	)
@@
 		(tags "rotary encoder")
 		(property "Reference" "SW10"
-			(at 2.8 -4.7 0)
+			(at 0.25 -5.5 0)
 			(layer "F.SilkS")
 			(effects
@@
 		)
 		(property "Value" "RotaryEncoder_Switch"
-			(at 7.5 10.4 0)
+			(at 8.25 10.4 0)
 			(layer "F.Fab")
 			(effects
@@
 		(tags "rotary encoder")
 		(property "Reference" "SW11"
-			(at 2.8 -4.7 0)
+			(at 0.25 -5.5 0)
 			(layer "F.SilkS")
 			(effects
@@
 		(layer "Edge.Cuts")
 	)
+	(gr_text "MACROMAX703"
+		(at 97 95 0)
+		(layer "F.SilkS")
+		(effects
+			(font
+				(size 1.5 1.5)
+				(thickness 0.3)
+				(bold yes)
+			)
+			(justify left bottom)
+		)
+	)
 	(segment
 		(start 116.19 82)
@@
 	)
 	(segment
-		(start 126.2 105.8)
-		(end 132.876598 105.8)
-		(width 0.2)
+		(start 134.424457 103.2105)
+		(end 140.7895 103.2105)
+		(width 0.127)
 		(layer "B.Cu")
 		(net "Net-(D6-A)")
 	)
 	(segment
-		(start 153.089662 103.247)
-		(end 161.19 95.146662)
-		(width 0.2)
+		(start 126 106)
+		(end 126.2495 105.7505)
+		(width 0.127)
 		(layer "B.Cu")
 		(net "Net-(D6-A)")
 	)
 	(segment
-		(start 126 106)
-		(end 126.2 105.8)
-		(width 0.2)
+		(start 126.2495 105.7505)
+		(end 131.884457 105.7505)
+		(width 0.127)
 		(layer "B.Cu")
 		(net "Net-(D6-A)")
 	)
 	(segment
-		(start 135.429598 103.247)
-		(end 145.526338 103.247)
-		(width 0.2)
+		(start 140.7895 103.2105)
+		(end 141.545457 102.454543)
+		(width 0.127)
 		(layer "B.Cu")
 		(net "Net-(D6-A)")
 	)
 	(segment
-		(start 147.081014 103.247)
-		(end 153.089662 103.247)
-		(width 0.2)
+		(start 161.19 95.095043)
+		(end 161.19 88.46)
+		(width 0.127)
 		(layer "B.Cu")
 		(net "Net-(D6-A)")
 	)
 	(segment
-		(start 145.526338 103.247)
-		(end 146.303676 102.469662)
-		(width 0.2)
+		(start 131.884457 105.7505)
+		(end 134.424457 103.2105)
+		(width 0.127)
 		(layer "B.Cu")
 		(net "Net-(D6-A)")
 	)
 	(segment
-		(start 132.876598 105.8)
-		(end 135.429598 103.247)
-		(width 0.2)
+		(start 153.074543 103.2105)
+		(end 161.19 95.095043)
+		(width 0.127)
 		(layer "B.Cu")
 		(net "Net-(D6-A)")
 	)
 	(segment
-		(start 161.19 95.146662)
-		(end 161.19 88.46)
-		(width 0.2)
+		(start 151.2495 102.454543)
+		(end 152.005457 103.2105)
+		(width 0.127)
 		(layer "B.Cu")
 		(net "Net-(D6-A)")
 	)
 	(segment
-		(start 146.303676 102.469662)
-		(end 147.081014 103.247)
-		(width 0.2)
+		(start 152.005457 103.2105)
+		(end 153.074543 103.2105)
+		(width 0.127)
+		(layer "B.Cu")
+		(net "Net-(D6-A)")
+	)
+	(segment
+		(start 141.545457 102.454543)
+		(end 151.2495 102.454543)
+		(width 0.127)
 		(layer "B.Cu")
 		(net "Net-(D6-A)")
