File: pcb/MacroMax703_pcb.kicad_sch (KiCad schematic)
At the start: 21 parts, among them SW1 SW_Push, SW10 RotaryEncoder_Switch, SW11 RotaryEncoder_Switch, SW2 SW_Push, SW3 SW_Push, SW4 SW_Push, SW5 SW_Push, SW6 SW_Push, SW7 SW_Push, SW8 SW_Push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

Commit message: update pcb and firmware
Other:
- moved on the sheet: SW11
Changed lines of the file:
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@@
 	(wire
 		(pts
-			(xy 189.23 104.14) (xy 175.26 104.14)
+			(xy 190.5 104.14) (xy 176.53 104.14)
 		)
 		(stroke
@@
 	(wire
 		(pts
-			(xy 173.99 109.22) (xy 173.99 63.5)
+			(xy 175.26 109.22) (xy 175.26 63.5)
 		)
 		(stroke
@@
 	(wire
 		(pts
-			(xy 175.26 104.14) (xy 175.26 64.77)
+			(xy 176.53 104.14) (xy 176.53 64.77)
 		)
 		(stroke
@@
 	(wire
 		(pts
-			(xy 189.23 109.22) (xy 173.99 109.22)
+			(xy 190.5 109.22) (xy 175.26 109.22)
 		)
 		(stroke
@@
 	(wire
 		(pts
-			(xy 175.26 64.77) (xy 116.84 64.77)
-		)
-		(stroke
-			(width 0)
-			(type default)
-		)
-	)
-	(wire
-		(pts
-			(xy 173.99 63.5) (xy 115.57 63.5)
+			(xy 176.53 64.77) (xy 116.84 64.77)
+		)
+		(stroke
+			(width 0)
+			(type default)
+		)
+	)
+	(wire
+		(pts
+			(xy 175.26 63.5) (xy 115.57 63.5)
 		)
 		(stroke
@@
 		)
 		(instances
-			(project "XAIO"
+			(project "MacroMax703_pcb"
 				(path "/5dc50f45-2023-4306-a658-a916799bf250"
 					(reference "D2")
@@
 		)
 		(instances
-			(project "XAIO"
+			(project "MacroMax703_pcb"
 				(path "/5dc50f45-2023-4306-a658-a916799bf250"
 					(reference "D1")
@@
 		)
 		(instances
-			(project "XAIO"
+			(project "MacroMax703_pcb"
 				(path "/5dc50f45-2023-4306-a658-a916799bf250"
 					(reference "D5")
@@
 		)
 		(instances
-			(project "XAIO"
+			(project "MacroMax703_pcb"
 				(path "/5dc50f45-2023-4306-a658-a916799bf250"
 					(reference "D9")
@@
 		)
 		(instances
-			(project "XAIO"
+			(project "MacroMax703_pcb"
 				(path "/5dc50f45-2023-4306-a658-a916799bf250"
 					(reference "SW8")
@@
 		)
 		(instances
-			(project "XAIO"
+			(project "MacroMax703_pcb"
 				(path "/5dc50f45-2023-4306-a658-a916799bf250"
 					(reference "SW5")
@@
 		)
 		(instances
-			(project "XAIO"
+			(project "MacroMax703_pcb"
 				(path "/5dc50f45-2023-4306-a658-a916799bf250"
 					(reference "#PWR04")
@@
 		)
 		(instances
-			(project "XAIO"
+			(project "MacroMax703_pcb"
 				(path "/5dc50f45-2023-4306-a658-a916799bf250"
 					(reference "SW3")
@@
 		)
 		(instances
-			(project "XAIO"
+			(project "MacroMax703_pcb"
 				(path "/5dc50f45-2023-4306-a658-a916799bf250"
 					(reference "SW10")
@@
 		)
 		(instances
-			(project "XAIO"
+			(project "MacroMax703_pcb"
 				(path "/5dc50f45-2023-4306-a658-a916799bf250"
 					(reference "D4")
@@
 		)
 		(instances
-			(project "XAIO"
+			(project "MacroMax703_pcb"
 				(path "/5dc50f45-2023-4306-a658-a916799bf250"
 					(reference "SW6")
@@
 		)
 		(instances
-			(project "XAIO"
+			(project "MacroMax703_pcb"
 				(path "/5dc50f45-2023-4306-a658-a916799bf250"
 					(reference "SW1")
@@
 		)
 		(instances
-			(project "XAIO"
+			(project "MacroMax703_pcb"
 				(path "/5dc50f45-2023-4306-a658-a916799bf250"
 					(reference "SW9")
@@
 	(symbol
 		(lib_id "power:GND")
-		(at 189.23 106.68 270)
+		(at 190.5 106.68 270)
 		(unit 1)
 		(body_style 1)
@@
 		(fields_autoplaced yes)
 		(property "Reference" "#PWR05"
-			(at 182.88 106.68 0)
+			(at 184.15 106.68 0)
 			(hide yes)
 			(show_name no)
@@
 		)
 		(property "Value" "GND"
-			(at 185.42 106.6799 90)
+			(at 186.69 106.6799 90)
 			(show_name no)
 			(do_not_autoplace no)
@@
 		)
 		(property "Footprint" ""
-			(at 189.23 106.68 0)
+			(at 190.5 106.68 0)
 			(hide yes)
 			(show_name no)
@@
 		)
 		(property "Datasheet" ""
-			(at 189.23 106.68 0)
+			(at 190.5 106.68 0)
 			(hide yes)
 			(show_name no)
@@
 		)
 		(property "Description" "Power symbol creates a global label with name \"GND\" , ground"
-			(at 189.23 106.68 0)
+			(at 190.5 106.68 0)
 			(hide yes)
 			(show_name no)
@@
 		)
 		(instances
-			(project "XAIO"
+			(project "MacroMax703_pcb"
 				(path "/5dc50f45-2023-4306-a658-a916799bf250"
 					(reference "#PWR05")
@@
 		)
 		(instances
-			(project "XAIO"
+			(project "MacroMax703_pcb"
 				(path "/5dc50f45-2023-4306-a658-a916799bf250"
 					(reference "SW4")
@@
 		)
 		(instances
-			(project "XAIO"
+			(project "MacroMax703_pcb"
 				(path "/5dc50f45-2023-4306-a658-a916799bf250"
 					(reference "#PWR02")
@@
 		)
 		(instances
-			(project "XAIO"
+			(project "MacroMax703_pcb"
 				(path "/5dc50f45-2023-4306-a658-a916799bf250"
 					(reference "D8")
@@
 		)
 		(instances
-			(project "XAIO"
+			(project "MacroMax703_pcb"
 				(path "/5dc50f45-2023-4306-a658-a916799bf250"
 					(reference "#PWR07")
@@
 		)
 		(instances
-			(project "XAIO"
+			(project "MacroMax703_pcb"
 				(path "/5dc50f45-2023-4306-a658-a916799bf250"
 					(reference "D6")
@@
 		)
 		(instances
-			(project "XAIO"
+			(project "MacroMax703_pcb"
 				(path "/5dc50f45-2023-4306-a658-a916799bf250"
 					(reference "SW2")
@@
 		)
 		(instances
-			(project "XAIO"
+			(project "MacroMax703_pcb"
 				(path "/5dc50f45-2023-4306-a658-a916799bf250"
 					(reference "D7")
@@
 	(symbol
 		(lib_id "Device:RotaryEncoder_Switch")
-		(at 196.85 106.68 0)
+		(at 198.12 106.68 0)
 		(unit 1)
 		(body_style 1)
@@
 		(fields_autoplaced yes)
 		(property "Reference" "SW11"
-			(at 196.85 96.52 0)
+			(at 198.12 96.52 0)
 			(show_name no)
 			(do_not_autoplace no)
@@
 		)
 		(property "Value" "RotaryEncoder_Switch"
-			(at 196.85 99.06 0)
+			(at 198.12 99.06 0)
 			(show_name no)
 			(do_not_autoplace no)
@@
 		)
 		(property "Footprint" "Rotary_Encoder:RotaryEncoder_Alps_EC11E-Switch_Vertical_H20mm"
-			(at 193.04 102.616 0)
+			(at 194.31 102.616 0)
 			(hide yes)
 			(show_name no)
@@
 		)
 		(property "Datasheet" ""
-			(at 196.85 100.076 0)
+			(at 198.12 100.076 0)
 			(hide yes)
 			(show_name no)
@@
 		)
 		(property "Description" "Rotary encoder, dual channel, incremental quadrate outputs, with switch"
-			(at 196.85 106.68 0)
+			(at 198.12 106.68 0)
 			(hide yes)
 			(show_name no)
@@
 		)
 		(instances
-			(project "XAIO"
+			(project "MacroMax703_pcb"
 				(path "/5dc50f45-2023-4306-a658-a916799bf250"
 					(reference "SW11")
@@
 		)
 		(instances
-			(project "XAIO"
+			(project "MacroMax703_pcb"
 				(path "/5dc50f45-2023-4306-a658-a916799bf250"
 					(reference "SW7")
@@
 		)
 		(instances
-			(project "XAIO"
+			(project "MacroMax703_pcb"
 				(path "/5dc50f45-2023-4306-a658-a916799bf250"
 					(reference "D3")
@@
 		)
 		(instances
-			(project "XAIO"
+			(project "MacroMax703_pcb"
 				(path "/5dc50f45-2023-4306-a658-a916799bf250"
 					(reference "U1")
